File: pcb/nfcxpansion.kicad_pcb (KiCad board)
At the start: 2 copper layers, 32 x 25.5 mm, 11 parts, among them U1 ST25DV04K-JFR6D3

Commit message: quick update, bom and stuff
Other:
- board text added: "NFC"
- board text added: "for Hackxpansion"
- board text added: "vejas.zip"
