File: pcb/nfcxpansion.kicad_sch (KiCad schematic)
At the start: 9 parts, among them U1 ST25DV04K-JFR6D3

Commit message: quick update, bom and stuff
Parts:
- C1: LCSC Part # (none) -> C5137486
- R1: LCSC Part # (none) -> C2906861
- R2: LCSC Part # (none) -> C140197
- R3: LCSC Part # (none) -> C324823
- R4, R5: LCSC Part # (none) -> C140158
- U1: LCSC Part # (none) -> C2654815
Connections:
- no-connect marks 2 -> 9
Other:
- moved on the sheet: R5
Changed lines of the file:
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@@
+	)
+	(junction
+		(at 82.55 68.58)
+		(diameter 0)
+		(color 0 0 0 0)
 	)
 	(junction
@@
 	)
 	(junction
-		(at 82.55 68.58)
-		(diameter 0)
-		(color 0 0 0 0)
-	)
-	(junction
 		(at 116.84 78.74)
 		(diameter 0)
@@
 	)
 	(no_connect
+		(at 153.67 83.82)
+	)
+	(no_connect
 		(at 110.49 66.04)
 	)
+	(no_connect
+		(at 181.61 86.36)
+	)
+	(no_connect
+		(at 181.61 78.74)
+	)
+	(no_connect
+		(at 181.61 83.82)
+	)
+	(no_connect
+		(at 153.67 86.36)
+	)
+	(no_connect
+		(at 153.67 81.28)
+	)
+	(no_connect
+		(at 181.61 81.28)
+	)
 	(wire
 		(pts
@@
 	(wire
 		(pts
+			(xy 82.55 63.5) (xy 82.55 68.58)
+		)
+		(stroke
+			(width 0)
+			(type default)
+		)
+	)
+	(wire
+		(pts
 			(xy 113.03 73.66) (xy 113.03 71.12)
 		)
@@
 		(pts
 			(xy 78.74 55.88) (xy 74.93 55.88)
-		)
-		(stroke
-			(width 0)
-			(type default)
-		)
-	)
-	(wire
-		(pts
-			(xy 82.55 60.96) (xy 82.55 55.88)
 		)
 		(stroke
@@
 			)
 		)
+		(property "LCSC Part #" "C324823"
+			(at 142.24 67.31 0)
+			(hide yes)
+			(show_name no)
+			(do_not_autoplace no)
+			(effects
+				(font
+					(size 1.27 1.27)
+				)
+			)
+		)
 		(pin "1"
 		)
@@
 			)
 		)
+		(property "LCSC Part #" "C2906861"
+			(at 115.57 60.96 0)
+			(hide yes)
+			(show_name no)
+			(do_not_autoplace no)
+			(effects
+				(font
+					(size 1.27 1.27)
+				)
+			)
+		)
 		(pin "1"
 		)
@@
 	(symbol
 		(lib_id "Device:R")
-		(at 82.55 64.77 0)
+		(at 82.55 59.69 0)
 		(unit 1)
 		(body_style 1)
@@
 		(dnp no)
 		(property "Reference" "R5"
-			(at 84.074 60.706 0)
+			(at 84.074 58.42 0)
 			(show_name no)
 			(do_not_autoplace no)
@@
 		)
 		(property "Value" "4.7k"
-			(at 84.074 63.246 0)
+			(at 84.074 60.96 0)
 			(show_name no)
 			(do_not_autoplace no)
@@
 		)
 		(property "Footprint" "Resistor_SMD:R_0402_1005Metric"
-			(at 80.772 64.77 90)
+			(at 80.772 59.69 90)
 			(hide yes)
 			(show_name no)
@@
 		)
 		(property "Datasheet" ""
-			(at 82.55 64.77 0)
+			(at 82.55 59.69 0)
 			(hide yes)
 			(show_name no)
@@
 		)
 		(property "Description" "Resistor"
-			(at 82.55 64.77 0)
+			(at 82.55 59.69 0)
+			(hide yes)
+			(show_name no)
+			(do_not_autoplace no)
+			(effects
+				(font
+					(size 1.27 1.27)
+				)
+			)
+		)
+		(property "LCSC Part #" "C140158"
+			(at 82.55 59.69 0)
 			(hide yes)
 			(show_name no)
@@
 		(lib_id "Device:R")
 		(at 74.93 59.69 0)
+		(mirror y)
 		(unit 1)
 		(body_style 1)
@@
 		(in_pos_files yes)
 		(dnp no)
-		(fields_autoplaced yes)
 		(property "Reference" "R4"
-			(at 77.47 58.4199 0)
+			(at 72.39 58.4199 0)
 			(show_name no)
 			(do_not_autoplace no)
@@
 		)
 		(property "Value" "4.7k"
-			(at 77.47 60.9599 0)
+			(at 72.39 60.9599 0)
 			(show_name no)
 			(do_not_autoplace no)
@@
 		)
 		(property "Footprint" "Resistor_SMD:R_0402_1005Metric"
-			(at 73.152 59.69 90)
+			(at 76.708 59.69 90)
 			(hide yes)
 			(show_name no)
@@
 		)
 		(property "Description" "Resistor"
+			(at 74.93 59.69 0)
+			(hide yes)
+			(show_name no)
+			(do_not_autoplace no)
+			(effects
+				(font
+					(size 1.27 1.27)
+				)
+			)
+		)
+		(property "LCSC Part #" "C140158"
 			(at 74.93 59.69 0)
 			(hide yes)
@@
 			)
 		)
+		(property "LCSC Part #" "C5137486"
+			(at 116.84 74.93 0)
+			(hide yes)
+			(show_name no)
+			(do_not_autoplace no)
+			(effects
+				(font
+					(size 1.27 1.27)
+				)
+			)
+		)
 		(pin "2"
 		)
@@
 			)
 		)
+		(property "LCSC Part #" "C2654815"
+			(at 97.79 71.12 0)
+			(hide yes)
+			(show_name no)
+			(do_not_autoplace no)
+			(effects
+				(font
+					(size 1.27 1.27)
+				)
+			)
+		)
 		(pin "5"
 		)
@@
 			(at 134.62 67.31 0)
 			(hide yes)
+			(show_name no)
+			(do_not_autoplace no)
+			(effects
+				(font
+					(size 1.27 1.27)
+				)
+			)
+		)
+		(property "LCSC Part #" "C140197"
+			(at 134.62 67.31 0)
+			(hide yes)
